Commit message: Having restored the coordinate of the car

File: src/robot_description/urdf/LiDAR.xacro (robot description, xacro)
@@ -9,8 +9,8 @@
             </geometry>
             <material name="grey"/>
-            <origin xyz="0 ${-lidar_radius} ${lidar_length / 2}" rpy="0 0 0" />
+            <origin xyz="${-lidar_radius} 0 ${lidar_length / 2}" rpy="0 0 0" />
         </visual>
         <xacro:cylinder_inertia m="0.1" r="${lidar_radius}" l="${lidar_length}"
-                    o_xyz="0 ${-lidar_radius} ${lidar_length / 2}" o_rpy="0 0 0"/>
+                    o_xyz="${-lidar_radius} 0 ${lidar_length / 2}" o_rpy="0 0 0"/>
     </link>
     <gazebo reference="laser_link">
@@ -18,5 +18,5 @@
             <visualize>true</visualize>
             <topic>/scan</topic>
-            <pose>0 0 0 0 0 ${pi/2}</pose>
+            <pose>0 0 0 0 0 0</pose>
             <update_rate>10</update_rate>
                 <ray>

File: src/robot_description/urdf/camera.xacro (robot description, xacro)
@@ -1,7 +1,5 @@
 <?xml version="1.0"?>
 <robot xmlns:xacro="http://www.ros.org/wiki/xacro">
-    <!-- This represents X -->
     <xacro:property name="camera_length" value="0.01"/>
-    <!-- This Y -->
     <xacro:property name="camera_width" value="0.1"/>
     <xacro:property name="camera_height" value="0.05"/>
@@ -30,5 +28,5 @@
         <parent link="base_link" />
         <child link="camera_link"/>
-        <origin xyz="0 ${(base_length + camera_length)/ 2} ${base_height / 2}" rpy="0 0 ${pi/2}"/>
+        <origin xyz="${(base_length + camera_length)/ 2} 0 ${base_height / 2}" rpy="0 0 0"/>
     </joint>
     <gazebo reference="camera_link">

File: src/robot_description/urdf/mobile_base.xacro (robot description, xacro)
@@ -9,5 +9,5 @@
         <visual>
             <geometry>
-                <box size="${base_width} ${base_length} ${base_height}" />
+                <box size="${base_length} ${base_width} ${base_height}" />
             </geometry>
             <origin xyz="0 0 ${base_height / 2}" rpy="0 0 0" />
@@ -16,9 +16,9 @@
         <collision>
             <geometry>
-                <box size="${base_width} ${base_length} ${base_height}" />
+                <box size="$${base_length} ${base_width} ${base_height}" />
             </geometry>
             <origin xyz="0 0 ${base_height / 2}" rpy="0 0 0" />
         </collision>
-        <xacro:box_inertia m="5.0" x="${base_width}" y="${base_length}" z="${base_height}"
+        <xacro:box_inertia m="5.0" x="${base_length}" y="${base_width}" z="${base_height}"
         o_xyz="0 0 ${base_height / 2}" o_rpy="0 0 0" />
     </link>
@@ -29,5 +29,5 @@
                     <cylinder radius="${wheel_radius}" length="${wheel_length}" />
                 </geometry>
-                <origin xyz="0 0 0" rpy="0 ${pi / 2.0} 0" />
+                <origin xyz="0 0 0" rpy="${pi / 2.0} 0 0" />
                 <material name="grey" />
             </visual>
@@ -65,18 +65,17 @@
         <parent link="base_link" />
         <child link="right_wheel_link" />
-        <origin xyz="${base_width / 2 + wheel_length / 2} ${-base_length / 5.0} 0" rpy="0 0 0" />
-        <axis xyz="1 0 0" />
+        <origin xyz="${-base_length / 5.0} ${base_width / 2 + wheel_length / 2} 0" rpy="0 0 0" />
+        <axis xyz="0 1 0" />
     </joint>
     <joint name="base_left_wheel_joint" type="continuous">
         <parent link="base_link" />
         <child link="left_wheel_link" />
-        <origin xyz="${-base_width / 2 + -wheel_length / 2} ${-base_length / 5.0} 0" rpy="0 0 0" />
-        <axis xyz="1 0 0" />
+        <origin xyz="${-base_length / 5.0} ${-base_width / 2 + -wheel_length / 2} 0" rpy="0 0 0" />
+        <axis xyz="0 1 0" />
     </joint>
     <joint name="base_caster_wheel_joint" type="fixed">
         <parent link="base_link" />
         <child link="caster_wheel_link" />
-        <origin xyz="0 ${base_length / 4.0} ${-wheel_radius / 2}" rpy="0 0 0" />
-        <axis xyz="1 0 0" />
+        <origin xyz="${base_length / 4.0} 0 ${-wheel_radius / 2}" rpy="0 0 0" />
     </joint>
     <joint name="base_joint" type="fixed">

File: src/robot_description/urdf/robot.urdf.xacro (robot description, xacro)
@@ -10,10 +10,10 @@
         <parent link="base_link" />
         <child link="arm_base_link" />
-        <origin xyz="0 ${base_length / 4} ${base_height}" rpy="0 0 0" />
+        <origin xyz="${base_length / 4} 0 ${base_height}" rpy="0 0 0" />
     </joint>
     <joint name="laser_joint" type="fixed">
         <parent link="base_link"/>
         <child link="laser_link"/>
-        <origin xyz="0 ${base_length / 2} ${base_height}" rpy="0 0 0"/>
+        <origin xyz="${base_length / 2} 0 ${base_height}" rpy="0 0 0"/>
     </joint>
 </robot>
